Commit message: Changed from pr2_lfd_vision to lfd_vision:   modified package name from pr2_lfd_vision to lfd_vision,   separated simulation stuff to the lfd_sim package,   works with PR2, Baxter, and other robots;

File: urdf/m100_clamp_mount.urdf.xacro (robot description, xacro)
@@ -24,5 +24,5 @@
         <origin xyz="0.0 0.0 0" rpy="0 0 0"/>
         <geometry>
-          <mesh filename="package://pr2_lfd_vision/meshes/m100_clamp_mount.stl" scale="0.01 0.01 0.01" />
+          <mesh filename="package://lfd_vision/meshes/m100_clamp_mount.stl" scale="0.01 0.01 0.01" />
         </geometry>
         <material name="gray">
@@ -33,5 +33,5 @@
         <origin xyz="0.0 0.0 0" rpy="0 0 0"/>
         <geometry>
-          <mesh filename="package://pr2_lfd_vision/meshes/m100_clamp_mount.stl" scale="0.01 0.01 0.01" />
+          <mesh filename="package://lfd_vision/meshes/m100_clamp_mount.stl" scale="0.01 0.01 0.01" />
         </geometry>
       </collision>

File: urdf/pr2_w_m100.urdf.xacro (robot description, xacro)
@@ -34,5 +34,5 @@
   <include filename="$(find pr2_description)/urdf/materials.urdf.xacro" />
   <!-- Sentis m100 and its mount -->
-  <include filename="$(find pr2_lfd_vision)/urdf/m100_clamp_mount.urdf.xacro" />
+  <include filename="$(find lfd_vision)/urdf/m100_clamp_mount.urdf.xacro" />
   <!-- Now we can start using the macros included above to define the actual PR2 -->
   <!-- The first use of a macro.  This one was defined in base.urdf.xacro above.
